File: kicad_hx711_tyny85/kicad_hx711_tyny85.kicad_pcb (KiCad board)
At the start: 2 copper layers, 15.2 x 19.2 mm, 17 parts, among them J1 Conn_01x03_Male, J2 Conn_01x04_Female, J3 Conn_01x01_Female, J4 Conn_01x01_Female, J5 Conn_01x01_Female, J6 Conn_01x01_Female, Q1 Q_PNP_BEC, U1 HX711, U2 ATtiny85V-10SU

Commit message: Split GND-AGND
Parts:
- added JP1: Jumper, void_foot:AnalogGND_jumper, B.Cu at (93.5, 80.8)
- moved J3 1.35 mm to (89.0, 76.2)
- moved C4 0.75 mm to (94.5, 86.8)
Connections:
- C2 pad 2: GND -> GNDA
- C3 pad 1: GND -> GNDA
- J2 pad 4: GND -> GNDA
- R2 pad 2: GND -> GNDA
- U1 pad 5: GND -> GNDA
Routing:
- net GND: track 51.3 -> 0.50 mm
- net GNDA: track 0.00 -> 18.6 mm
- net INNA: track 8.03 -> 9.80 mm
- net RST: track 1.89 -> 3.34 mm
